Commit message: convert to .obj .mtl w/ texture maps

File: franka_description_pybullet/robots/common/franka_hand.xacro (robot description, xacro)
@@ -26,5 +26,5 @@
       <visual>
         <geometry>
-          <mesh filename="$(cwd)/../../meshes/visual/finger.dae" />
+          <mesh filename="$(cwd)/../../meshes/visual/finger.obj" />
         </geometry>
       </visual>
@@ -65,5 +65,5 @@
         <origin xyz="0 0 0" rpy="0 0 ${pi}" />
         <geometry>
-          <mesh filename="$(cwd)/../../meshes/visual/finger.dae" />
+          <mesh filename="$(cwd)/../../meshes/visual/finger.obj" />
         </geometry>
       </visual>

File: franka_description_pybullet/robots/common/utils.xacro (robot description, xacro)
@@ -38,5 +38,5 @@
       <visual>
         <geometry>
-          <mesh filename="$(cwd)/../../meshes/visual/${name}.dae" />
+          <mesh filename="$(cwd)/../../meshes/visual/${name}.obj" />
         </geometry>
       </visual>

Commit message: fix texturing

File: franka_description_pybullet/robots/common/franka_hand.xacro (robot description, xacro)
@@ -28,4 +28,7 @@
           <mesh filename="$(cwd)/../../meshes/visual/finger.obj" />
         </geometry>
+        <material name="panda_white">
+          <color rgba="1. 1. 1. 1."/>
+        </material>
       </visual>
       <!-- screw mount -->
@@ -67,4 +70,7 @@
           <mesh filename="$(cwd)/../../meshes/visual/finger.obj" />
         </geometry>
+        <material name="panda_white">
+          <color rgba="1. 1. 1. 1."/>
+        </material>
       </visual>
       <!-- screw mount -->

File: franka_description_pybullet/robots/common/utils.xacro (robot description, xacro)
@@ -40,4 +40,7 @@
           <mesh filename="$(cwd)/../../meshes/visual/${name}.obj" />
         </geometry>
+        <material name="panda_white">
+          <color rgba="1. 1. 1. 1."/>
+        </material>
       </visual>
       <collision>
