Commit message: changed mesh path in urdf

File: franka_description_pybullet/robots/fr3/fr3_pybullet.urdf (robot description, URDF)
Before this commit: robot fr3, 22 links, 21 joints
Links:
- link fr3_hand: geometry collision mesh filename=./franka_description_pybullet/meshes/collision/hand.stl; visual mesh filename=./franka_description_pybullet/meshes/visual/hand.obj
- link fr3_leftfinger: geometry collision box size=17.5e-3 15.2e-3 18.5e-3; collision box size=17.5e-3 7e-3 23.5e-3
- link fr3_link0: geometry collision mesh filename=./franka_description_pybullet/meshes/collision/link0.stl; visual mesh filename=./franka_description_pybullet/meshes/visual/link0.obj
- link fr3_link1: geometry collision mesh filename=./franka_description_pybullet/meshes/collision/link1.stl; visual mesh filename=./franka_description_pybullet/meshes/visual/link1.obj
- link fr3_link2: geometry collision mesh filename=./franka_description_pybullet/meshes/collision/link2.stl; visual mesh filename=./franka_description_pybullet/meshes/visual/link2.obj
- link fr3_link3: geometry collision mesh filename=./franka_description_pybullet/meshes/collision/link3.stl; visual mesh filename=./franka_description_pybullet/meshes/visual/link3.obj
- link fr3_link4: geometry collision mesh filename=./franka_description_pybullet/meshes/collision/link4.stl; visual mesh filename=./franka_description_pybullet/meshes/visual/link4.obj
- link fr3_link5: geometry collision mesh filename=./franka_description_pybullet/meshes/collision/link5.stl; visual mesh filename=./franka_description_pybullet/meshes/visual/link5.obj
- link fr3_link6: geometry collision mesh filename=./franka_description_pybullet/meshes/collision/link6.stl; visual mesh filename=./franka_description_pybullet/meshes/visual/link6.obj
- link fr3_link7: geometry collision mesh filename=./franka_description_pybullet/meshes/collision/link7.stl; visual mesh filename=./franka_description_pybullet/meshes/visual/link7.obj
- link fr3_rightfinger: geometry collision box size=17.5e-3 15.2e-3 18.5e-3; collision box size=17.5e-3 7e-3 23.5e-3
